Commit message: feat: add IsaacLab policy instance in d1, and fix urdf of d1

File: urdfs/d1_description/urdf/robot.urdf (robot description, URDF)
Before this commit: robot d1_description, 24 links, 23 joints
Links:
- link FL_calf: geometry collision box size=0.24 0.04 0.05; visual mesh filename=package://d1h_description/meshes/L_calf.STL
- link FL_foot: geometry collision cylinder length=0.04 radius=0.087; visual mesh filename=package://d1h_description/meshes/L_foot.STL
- link FL_hip: geometry visual mesh filename=package://d1h_description/meshes/L_hip.STL
- link FL_thigh: geometry collision box size=0.26 0.09 0.05; visual mesh filename=package://d1h_description/meshes/L_thigh.STL
- link FR_calf: geometry collision box size=0.24 0.04 0.05; visual mesh filename=package://d1h_description/meshes/R_calf.STL
- link FR_foot: geometry collision cylinder length=0.04 radius=0.087; visual mesh filename=package://d1h_description/meshes/R_foot.STL
- link FR_hip: geometry visual mesh filename=package://d1h_description/meshes/R_hip.STL
- link FR_thigh: geometry collision box size=0.26 0.09 0.05; visual mesh filename=package://d1h_description/meshes/R_thigh.STL
- link F_base_link: geometry collision box size=0.275 0.15 0.175; collision box size=0.31 0.12 0.06
- link F_docking_link: geometry collision box size=0.0851 0.15 0.175; visual mesh filename=package://d1h_description/meshes/docking_Link.STL
- link F_funtion_link: geometry collision box size=0.0495 0.15 0.175; visual mesh filename=package://d1h_description/meshes/funtion_Link.STL
- link RL_calf: geometry collision box size=0.24 0.04 0.05; visual mesh filename=package://d1h_description/meshes/L_calf.STL
- link RL_foot: geometry collision cylinder length=0.04 radius=0.087; visual mesh filename=package://d1h_description/meshes/L_foot.STL
- link RL_hip: geometry visual mesh filename=package://d1h_description/meshes/L_hip.STL
- link RL_thigh: geometry collision box size=0.26 0.09 0.05; visual mesh filename=package://d1h_description/meshes/L_thigh.STL
- link RR_calf: geometry collision box size=0.24 0.04 0.05; visual mesh filename=package://d1h_description/meshes/R_calf.STL
- link RR_foot: geometry collision cylinder length=0.04 radius=0.087; visual mesh filename=package://d1h_description/meshes/R_foot.STL
- link RR_hip: geometry visual mesh filename=package://d1h_description/meshes/R_hip.STL
- link RR_thigh: geometry collision box size=0.26 0.09 0.05; visual mesh filename=package://d1h_description/meshes/R_thigh.STL
- link R_base_link: geometry collision box size=0.275 0.15 0.175; collision box size=0.31 0.12 0.06
- link R_docking_link: geometry collision box size=0.0851 0.15 0.175; visual mesh filename=package://d1h_description/meshes/docking_Link.STL
- link R_funtion_link: geometry collision box size=0.0495 0.15 0.175; visual mesh filename=package://d1h_description/meshes/funtion_Link.STL
