Commit message: Add commanded body-height RL controller for d1cargo (key 4)
Variable flat-ground body height: 4th command channel (base_height) with
keyboard q/e, plus the rl_height_cargo config, obs/command loading, and the
cargo mujoco model.

File: urdfs/d1_description/urdf/robot_cargo.urdf (robot description, URDF)
Before this commit: robot d1_description, 25 links, 24 joints
Links:
- link cargo_box: geometry collision box size=0.30 0.26 0.20; visual box size=0.30 0.26 0.20
Joints:
- joint cargo_box_joint: origin xyz=0 0 -0.01 rpy=0 0 0 -> xyz=0 0 -0.03 rpy=0 0 0
