Commit message: d1cargo: flip rear module 180 for back-to-back symmetry, update height policy
Rotate the rear d1h module 180 about z in both URDF and MuJoCo model so it matches the real back-to-back assembly, recenter base inertia, and deploy the retrained symmetric height policy.

File: urdfs/d1_description/urdf/robot_cargo.urdf (robot description, URDF)
Before this commit: robot d1_description, 25 links, 24 joints
Joints:
- joint R_base_joint: origin xyz=-0.36 0 0 rpy=0 0 0 -> xyz=-0.36 0 0 rpy=0 0 3.14159
- joint R_docking_joint: origin xyz=0.187 0 0 rpy=0 0 3.14159 -> xyz=-0.187 0 0 rpy=0 0 0
- joint R_funtion_joint: origin xyz=-0.1545 0 0 rpy=0 0 3.14159 -> xyz=0.1545 0 0 rpy=0 0 0
