Commit message: fix urdf bug

File: urdfs/d1_description/urdf/robot_cargo_out.urdf (robot description, URDF)
Before this commit: robot d1_description, 25 links, 24 joints
Joints:
- joint F_docking_joint: origin xyz=-0.187 0 0 rpy=0 0 0 -> xyz=0.187 0 0 rpy=0 0 3.14159
- joint F_funtion_joint: origin xyz=0.1545 0 0 rpy=0 0 0 -> xyz=-0.1545 0 0 rpy=0 0 3.14159
- joint R_docking_joint: origin xyz=-0.187 0 0 rpy=0 0 0 -> xyz=0.187 0 0 rpy=0 0 3.14159
- joint R_funtion_joint: origin xyz=0.1545 0 0 rpy=0 0 0 -> xyz=-0.1545 0 0 rpy=0 0 3.14159

Commit message: update model to mower

File: urdfs/d1_description/urdf/robot_cargo_out.urdf (robot description, URDF)
Before this commit: robot d1_description, 25 links, 24 joints
Links:
- removed link cargo_box
- added link mower, mass 22.872; collision mesh filename=package://d1_description/meshes/mower.STL; visual mesh filename=package://d1_description/meshes/mower.STL
- link FL_calf: mass 0.46345045 -> 0.61004; geometry collision box size=0.3 0.04 0.05; visual mesh filename=package://d1h_description/meshes/L_calf.STL
- link FL_foot: mass 1.6631 -> 1.75470
- link FL_hip: mass 1.69464273 -> 1.86700
- link FL_thigh: mass 2.55232244 -> 2.81160; geometry collision box size=0.3 0.09 0.05; visual mesh filename=package://d1h_description/meshes/L_thigh.STL
- link FR_calf: mass 0.46345511 -> 0.61004; geometry collision box size=0.3 0.04 0.05; visual mesh filename=package://d1h_description/meshes/R_calf.STL
- link FR_foot: mass 1.6631 -> 1.75470
- link FR_hip: mass 1.69464279 -> 1.86700
- link FR_thigh: mass 2.55232278 -> 2.81160; geometry collision box size=0.3 0.09 0.05; visual mesh filename=package://d1h_description/meshes/R_thigh.STL
- link F_base_link: mass 8.44614222 -> 9.158; geometry collision box size=0.275 0.15 0.18; collision box size=0.35 0.15 0.1
- link F_docking_link: mass 2.20153411 -> 1.1043; geometry collision box size=0.0495 0.15 0.175; visual mesh filename=package://d1h_description/meshes/docking_Link.STL
- link F_funtion_link: mass 0.67772 -> 0.7859; geometry collision box size=0.0495 0.15 0.18; visual mesh filename=package://d1h_description/meshes/funtion_Link.STL
- link RL_calf: mass 0.46345045 -> 0.61004; geometry collision box size=0.3 0.04 0.05; visual mesh filename=package://d1h_description/meshes/L_calf.STL
- link RL_foot: mass 1.6631 -> 1.75470
- link RL_hip: mass 1.69464273 -> 1.86700
- link RL_thigh: mass 2.55232244 -> 2.81160; geometry collision box size=0.3 0.09 0.05; visual mesh filename=package://d1h_description/meshes/L_thigh.STL
- link RR_calf: mass 0.46345511 -> 0.61004; geometry collision box size=0.3 0.04 0.05; visual mesh filename=package://d1h_description/meshes/R_calf.STL
- link RR_foot: mass 1.6631 -> 1.75470
- link RR_hip: mass 1.69464279 -> 1.86700
- link RR_thigh: mass 2.55232278 -> 2.81160; geometry collision box size=0.3 0.09 0.05; visual mesh filename=package://d1h_description/meshes/R_thigh.STL
- link R_base_link: mass 8.44614222 -> 9.158; geometry collision box size=0.275 0.15 0.18; collision box size=0.35 0.15 0.1
- link R_docking_link: mass 2.20153411 -> 1.1043; geometry collision box size=0.0495 0.15 0.175; visual mesh filename=package://d1h_description/meshes/docking_Link.STL
- link R_funtion_link: mass 0.67772 -> 0.7859; geometry collision box size=0.0495 0.15 0.18; visual mesh filename=package://d1h_description/meshes/funtion_Link.STL
Joints:
- removed joint cargo_box_joint
- added joint mower_joint: type fixed, parent base_link, child mower, origin xyz=0 0 -0.02 rpy=0 0 0
- joint FL_calf_joint: limit lower=-2.775 upper=-0.855 effort=80 velocity=20 -> lower=-2.72 upper=-0.85 effort=80 velocity=20
- joint FL_foot_joint: limit lower=-1000000.0 upper=1000000.0 effort=12 velocity=30.0 -> lower=-31415926 upper=31415926 effort=12 velocity=30.0
- joint FR_calf_joint: limit lower=-2.775 upper=-0.855 effort=80 velocity=20 -> lower=-2.72 upper=-0.85 effort=80 velocity=20
- joint FR_foot_joint: limit lower=-1000000.0 upper=1000000.0 effort=12 velocity=30.0 -> lower=-31415926 upper=31415926 effort=12 velocity=30.0
- joint F_base_joint: origin xyz=0.36 0 0 rpy=0 0 3.14159 -> xyz=0.553 0 0 rpy=0 0 3.14159
- joint RL_calf_joint: limit lower=-2.775 upper=-0.855 effort=80 velocity=20 -> lower=-2.72 upper=-0.85 effort=80 velocity=20
- joint RL_foot_joint: limit lower=-1000000.0 upper=1000000.0 effort=12 velocity=30.0 -> lower=-31415926 upper=31415926 effort=12 velocity=30.0
- joint RR_calf_joint: limit lower=-2.775 upper=-0.855 effort=80 velocity=20 -> lower=-2.72 upper=-0.85 effort=80 velocity=20
- joint RR_foot_joint: limit lower=-1000000.0 upper=1000000.0 effort=12 velocity=30.0 -> lower=-31415926 upper=31415926 effort=12 velocity=30.0
- joint R_base_joint: origin xyz=-0.36 0 0 rpy=0 0 0 -> xyz=-0.553 0 0 rpy=0 0 0

File: urdfs/d1_description/xacro/robot_cargo_out.xacro (robot description, xacro)
@@ -2,7 +2,7 @@
 <!-- d1cargo "out" (<>) variant: original robot.xacro is kept untouched.
      Matches urdf/robot_cargo_out.urdf and mujoco/robot_cargo_out.xml:
-       - central cargo box (0.30 x 0.26 x 0.20, 6 kg) fixed under base_link
-       - modules moved apart: +-0.1875 -> +-0.36 to make room for the box
-       - F module yawed 180deg (yaw=3.14159) -> hips inboard at +-0.2655,
+       - central mower payload (mesh mower.STL, 22.872 kg), lowered 2cm (mower_joint z=-0.02)
+       - modules moved apart: +-0.1875 -> +-0.553 (widened +16cm/side to seat mower docking)
+       - F module yawed 180deg (yaw=3.14159) -> hips inboard at +-0.4585,
          knees point outward = "<>" stance; R module not rotated
      Uses single_robot_out.xacro (yaw param + pi-compensated funtion/docking). -->
@@ -27,28 +27,32 @@
         </inertial>
     </link>
-    <!-- central cargo box between the two modules -->
-    <link name="cargo_box">
+    <!-- central mower payload between the two modules (SolidWorks 负载框-割草机版, 22.872 kg).
+         mesh frame == base_link frame, so the fixed joint stays at the origin. -->
+    <link name="mower">
         <visual>
             <origin rpy="0 0 0" xyz="0 0 0"/>
             <geometry>
-                <box size="0.30 0.26 0.20"/>
+                <mesh filename="package://d1_description/meshes/mower.STL"/>
             </geometry>
+            <material name="">
+                <color rgba="0.75294 0.75294 0.75294 1"/>
+            </material>
         </visual>
         <collision>
             <origin rpy="0 0 0" xyz="0 0 0"/>
             <geometry>
-                <box size="0.30 0.26 0.20"/>
+                <mesh filename="package://d1_description/meshes/mower.STL"/>
             </geometry>
         </collision>
         <inertial>
-            <mass value="6.0"/>
-            <origin rpy="0 0 0" xyz="0 0 0"/>
-            <inertia ixx="0.0538" ixy="0" ixz="0" iyy="0.065" iyz="0" izz="0.0788"/>
+            <mass value="22.872"/>
+            <origin rpy="0 0 0" xyz="-0.0099654 -0.00019956 0.0801"/>
+            <inertia ixx="0.59821" ixy="0.0059593" ixz="-0.0049803" iyy="1.2381" iyz="3.5606e-05" izz="1.1939"/>
         </inertial>
     </link>
-    <joint name="cargo_box_joint" type="fixed">
-        <origin rpy="0 0 0" xyz="0 0 -0.03"/>
+    <joint name="mower_joint" type="fixed">
+        <origin rpy="0 0 0" xyz="0 0 -0.02"/>
         <parent link="base_link"/>
-        <child link="cargo_box"/>
+        <child link="mower"/>
     </joint>
     <link name="imu_link">
@@ -78,5 +82,5 @@
     </joint>
     <!-- F module flipped 180deg (yaw) -> "<>" outward stance; R not rotated -->
-    <xacro:single_robot_out name="F" x_offset="0.36" yaw="3.14159"/>
-    <xacro:single_robot_out name="R" x_offset="-0.36"/>
+    <xacro:single_robot_out name="F" x_offset="0.553" yaw="3.14159"/>
+    <xacro:single_robot_out name="R" x_offset="-0.553"/>
 </robot>

File: urdfs/d1_description/xacro/single_robot_out.xacro (robot description, xacro)
@@ -14,7 +14,7 @@
         <link name="${name}_base_link">
             <inertial>
-                <origin xyz="0.04005271 0.00019692 -0.02084955" rpy="0 0 0" />
-                <mass value="8.44614222" />
-                <inertia ixx="0.07256618" ixy="0.00023603" ixz="-0.00688763" iyy="0.11587953" iyz="3.472e-05" izz="0.11697399"/>
+                <origin xyz="0.03074 0.00016 -0.03314" rpy="0 0 0" />
+                <mass value="9.158" />
+                <inertia ixx="0.073416" ixy="0.00014675" ixz="-0.0079314" iyy="0.12672" iyz="1.9414e-05" izz="0.11933"/>
             </inertial>
             <visual>
@@ -30,5 +30,5 @@
                 <origin xyz="0 0 0" rpy="0 0 0" />
                 <geometry>
-                    <box size="0.275 0.15 0.175"/>
+                    <box size="0.275 0.15 0.18"/>
                 </geometry>
             </collision>
@@ -36,5 +36,5 @@
                 <origin xyz="0 0 -0.12" rpy="0 0 0" />
                 <geometry>
-                    <box size="0.31 0.12 0.06"/>
+                    <box size="0.35 0.15 0.1"/>
                 </geometry>
             </collision>
@@ -48,7 +48,7 @@
         <link name="${name}_funtion_link">
             <inertial>
-                <origin xyz="0.01321944 0.0 0.00563897" rpy="0 0 0" />
-                <mass value="0.67772" />
-                <inertia ixx="0.0046602" ixy="-4.1631E-09" ixz="4.51E-05" iyy="0.0017478" iyz="8e-08" izz="0.0031524" />
+                <origin xyz="-0.02031 -0.00001 0.00546" rpy="0 0 0" />
+                <mass value="0.7859" />
+                <inertia ixx="0.005595" ixy="0.0" ixz="-4.5e-05" iyy="0.002202" iyz="0.0" izz="0.003725" />
             </inertial>
             <visual>
@@ -64,5 +64,5 @@
                 <origin xyz="0.008 0 0" rpy="0 0 0" />
                 <geometry>
-                    <box size="0.0495 0.15 0.175"/>
+                    <box size="0.0495 0.15 0.18"/>
                 </geometry>
             </collision>
@@ -77,7 +77,7 @@
         <link name="${name}_docking_link">
             <inertial>
-                <origin xyz="0.01527894 0.00855247 0.00284739" rpy="0 0 0" />
-                <mass value="2.20153411" />
-                <inertia ixx="0.01876158" ixy="0.00036494" ixz="6.869e-05" iyy="0.00631988" iyz="0.0001511" izz="0.01358894"/>
+                <origin xyz="0.01167 0.01142 0.00562" rpy="0 0 0" />
+                <mass value="1.1043" />
+                <inertia ixx="0.007968" ixy="0.000348" ixz="1.4e-05" iyy="0.002634" iyz="-1.7e-05" izz="0.005995"/>
             </inertial>
             <visual>
@@ -93,5 +93,5 @@
                 <origin xyz="0.0065 0 0" rpy="0 0 0" />
                 <geometry>
-                    <box size="0.0851 0.15 0.175"/>
+                    <box size="0.0495 0.15 0.175"/>
                 </geometry>
             </collision>
@@ -106,7 +106,7 @@
         <link name="${name}L_hip">
             <inertial>
-                <origin xyz="-0.01814352 -7.96e-06 -0.09365134" rpy="0 0 0" />
-                <mass value="1.69464273" />
-                <inertia ixx="0.00379266" ixy="-1.1e-07" ixz="-2.452e-05" iyy="0.00276068" iyz="3.09e-06" izz="0.00214485" />
+                <origin xyz="-0.01567766 -0.00005214 -0.09306106" rpy="0 0 0" />
+                <mass value="1.86700" />
+                <inertia ixx="0.004561" ixy="-0.00000066" ixz="-0.00004876" iyy="0.0034067" iyz="-0.00000146" izz="0.0026097" />
             </inertial>
             <visual>
@@ -125,5 +125,5 @@
             <child link="${name}L_hip" />
             <axis xyz="0 0 1" />
-            <dynamics damping="0" friction="0"/>
+            <dynamics damping="0.2346" friction="0.943"/>
             <limit effort="80" lower="-0.7853981633974483" upper="0.7853981633974483" velocity="20"/>
         </joint>
@@ -131,7 +131,7 @@
         <link name="${name}L_thigh">
             <inertial>
-                <origin xyz="0.02895091 0.00356333 -0.02811556" rpy="0 0 0" />
-                <mass value="2.55232244" />
-                <inertia ixx="0.00426053" ixy="-0.00133627" ixz="-0.00212533" iyy="0.01734276" iyz="-0.00029985" izz="0.01796394" />
+                <origin xyz="0.03137855 0.00371524 0.06475758" rpy="0 0 0" />
+                <mass value="2.81160" />
+                <inertia ixx="0.00486852" ixy="-0.00149035" ixz="-0.00234028" iyy="0.0203762" iyz="-0.00032034" izz="0.02095408" />
             </inertial>
             <visual>
@@ -147,5 +147,5 @@
                 <origin xyz="0.06 0.02 0" rpy="0 0 0.2617993877991494" />
                 <geometry>
-                    <box size="0.26 0.09 0.05"/>
+                    <box size="0.3 0.09 0.05"/>
                 </geometry>
             </collision>
@@ -156,5 +156,5 @@
             <child link="${name}L_thigh" />
             <axis xyz="0 0 1" />
-            <dynamics damping="0" friction="0"/>
+            <dynamics damping="0.2346" friction="0.943"/>
             <limit effort="80" lower="-1.8325957145940461" upper="3.4033920413889422" velocity="20"/>
         </joint>
@@ -162,7 +162,7 @@
         <link name="${name}L_calf">
             <inertial>
-                <origin xyz="0.12506267 0.00606587 0.00312587" rpy="0 0 0" />
-                <mass value="0.46345045" />
-                <inertia ixx="0.00023821" ixy="0.00034272" ixz="-0.00014416" iyy="0.00488539" iyz="3.83e-06" izz="0.00493944" />
+                <origin xyz="0.12683437 0.01137531 0.00486771" rpy="0 0 0" />
+                <mass value="0.61004" />
+                <inertia ixx="0.00034763" ixy="0.00045139" ixz="-0.00028304" iyy="0.0068336" iyz="0.00001004" izz="0.00692927" />
             </inertial>
             <visual>
@@ -178,5 +178,5 @@
                 <origin xyz="0.15 0.01 0" rpy="0 0 -0.08" />
                 <geometry>
-                    <box size="0.24 0.04 0.05"/>
+                    <box size="0.3 0.04 0.05"/>
                 </geometry>
             </collision>
@@ -187,13 +187,13 @@
             <child link="${name}L_calf" />
             <axis xyz="0 0 1" />
-            <dynamics damping="0" friction="0"/>
-            <limit effort="80" lower="-2.775" upper="-0.855" velocity="20"/>
+            <dynamics damping="0.2346" friction="0.943"/>
+            <limit effort="80" lower="-2.72" upper="-0.85" velocity="20"/>
         </joint>
         <!-- Left wheel link -->
         <link name="${name}L_foot">
             <inertial>
-                <origin xyz="-2.82e-06 0.0 -0.00091845" rpy="0 0 0" />
-                <mass value="1.6631" />
-                <inertia ixx="0.00397025" ixy="2.224e-05" ixz="2.1e-07" iyy="0.00395149" iyz="2e-07" izz="0.00760863" />
+                <origin xyz="-0.00001088 0.00000319 0.02475" rpy="0 0 0" />
+                <mass value="1.75470" />
+                <inertia ixx="0.00414743" ixy="-0.00000091" ixz="0.00000144" iyy="0.00415057" iyz="0.00000073" izz="0.0078035" />
             </inertial>
             <visual>
@@ -218,13 +218,13 @@
             <child link="${name}L_foot" />
             <axis xyz="0 0 1" />
-            <dynamics damping="0" friction="0"/>
-            <limit effort="12" lower="-1000000.0" upper="1000000.0" velocity="30.0"/>
+            <dynamics damping="0.5" friction="0.0"/>
+            <limit effort="12" lower="-31415926" upper="31415926" velocity="30.0"/>
         </joint>
         <!-- Right hip link -->
         <link name="${name}R_hip">
             <inertial>
-                <origin xyz="0.01814352 -8e-06 -0.09365134" rpy="0 0 0" />
-                <mass value="1.69464279" />
-                <inertia ixx="0.00379266" ixy="1.1e-07" ixz="2.452e-05" iyy="0.00276068" iyz="3.09e-06" izz="0.00214485" />
+                <origin xyz="0.01567834 -0.00005214 -0.09306094" rpy="0 0 0" />
+                <mass value="1.86700" />
+                <inertia ixx="0.004561" ixy="0.00000066" ixz="0.00004878" iyy="0.0034067" iyz="-0.00000146" izz="0.0026097" />
             </inertial>
             <visual>
@@ -243,5 +243,5 @@
             <child link="${name}R_hip" />
             <axis xyz="0 0 1" />
-            <dynamics damping="0" friction="0"/>
+            <dynamics damping="0.2346" friction="0.943"/>
             <limit effort="80" lower="-0.7853981633974483" upper="0.7853981633974483" velocity="20"/>
         </joint>
@@ -249,7 +249,7 @@
         <link name="${name}R_thigh">
             <inertial>
-                <origin xyz="0.0291816 0.00370278 0.02811568" rpy="0 0 0" />
-                <mass value="2.55232278" />
-                <inertia ixx="0.00427405" ixy="-0.00133225" ixz="0.00213801" iyy="0.01729241" iyz="0.00030751" izz="0.01792714" />
+                <origin xyz="0.03137957 0.00371556 -0.06475707" rpy="0 0 0" />
+                <mass value="2.81160" />
+                <inertia ixx="0.00486845" ixy="-0.00149037" ixz="0.00234002" iyy="0.02037619" iyz="0.00032032" izz="0.02095416" />
             </inertial>
             <visual>
@@ -265,5 +265,5 @@
                 <origin xyz="0.06 0.02 0" rpy="0 0 0.2617993877991494" />
                 <geometry>
-                    <box size="0.26 0.09 0.05"/>
+                    <box size="0.3 0.09 0.05"/>
                 </geometry>
             </collision>
@@ -274,5 +274,5 @@
             <child link="${name}R_thigh" />
             <axis xyz="0 0 1" />
-            <dynamics damping="0" friction="0"/>
+            <dynamics damping="0.2346" friction="0.943"/>
             <limit effort="80" lower="-1.8325957145940461" upper="3.4033920413889422" velocity="20"/>
         </joint>
@@ -280,7 +280,7 @@
         <link name="${name}R_calf">
             <inertial>
-                <origin xyz="0.12506359 0.00606606 -0.0031258" rpy="0 0 0" />
-                <mass value="0.46345511" />
-                <inertia ixx="0.00023821" ixy="0.00034271" ixz="0.00014415" iyy="0.00488543" iyz="-3.83e-06" izz="0.00493948" />
+                <origin xyz="0.12683435 0.01137538 -0.00486802" rpy="0 0 0" />
+                <mass value="0.61004" />
+                <inertia ixx="0.00034764" ixy="0.00045139" ixz="0.00028307" iyy="0.0068336" iyz="-0.00001004" izz="0.00692927" />
             </inertial>
             <visual>
@@ -296,5 +296,5 @@
                 <origin xyz="0.15 0.01 0" rpy="0 0 -0.08" />
                 <geometry>
-                    <box size="0.24 0.04 0.05"/>
+                    <box size="0.3 0.04 0.05"/>
                 </geometry>
             </collision>
@@ -305,13 +305,13 @@
             <child link="${name}R_calf" />
             <axis xyz="0 0 1" />
-            <dynamics damping="0" friction="0"/>
-            <limit effort="80" lower="-2.775" upper="-0.855" velocity="20"/>
+            <dynamics damping="0.2346" friction="0.943"/>
+            <limit effort="80" lower="-2.72" upper="-0.85" velocity="20"/>
         </joint>
         <!-- Right wheel link -->
         <link name="${name}R_foot">
             <inertial>
-                <origin xyz="-2.78e-06 0.0 0.00091859" rpy="0 0 0" />
-                <mass value="1.6631" />
-                <inertia ixx="0.00397018" ixy="2.222e-05" ixz="-2.1e-07" iyy="0.00395159" iyz="-2e-07" izz="0.00760867" />
+                <origin xyz="0.0000105 0.0000048 -0.02475" rpy="0 0 0" />
+                <mass value="1.75470" />
+                <inertia ixx="0.00414978" ixy="-0.00000164" ixz="0.00000051" iyy="0.00414822" iyz="0.00000155" izz="0.0078035" />
             </inertial>
             <visual>
@@ -336,6 +336,6 @@
             <child link="${name}R_foot" />
             <axis xyz="0 0 1" />
-            <dynamics damping="0" friction="0"/>
-            <limit effort="12" lower="-1000000.0" upper="1000000.0" velocity="30.0"/>
+            <dynamics damping="0.5" friction="0.0"/>
+            <limit effort="12" lower="-31415926" upper="31415926" velocity="30.0"/>
         </joint>
     </xacro:macro>
